File: Hardware/Sensor/Sensor Completed Project Folder/DCA_USMR_Sens/DCA_USMR_Sens.kicad_pcb (KiCad board)
At the start: 4 copper layers, 19 parts, among them U1 LM555xM, U2 MAX4528CSA+, U3 MAX4528CSA+, U4 SN74AHC1G04DBVR, U5 LM193DR

Commit message: Sensor Rev1.1
Rev1.1
Parts:
- added C10: 1u, Capacitor_SMD:C_0402_1005Metric, F.Cu at (237.1, 157.9)
- added C9: 10uF, Capacitor_SMD:C_0402_1005Metric, F.Cu at (234.0, 142.6)
- added D1: 1Vf, DIOAD835W50L444D203:DIOAD835W50L444D203, F.Cu at (241.1, 139.3)
- added R5: 220, Resistor_SMD:R_0402_1005Metric, F.Cu at (234.5, 140.6)
- R3: value 2.2k -> 2.7k
- R4: value 22k -> 560
- moved C5 97.5 mm to (241.0, 154.1)
- moved C6 97.5 mm to (240.5, 144.4)
- moved C7 97.5 mm to (233.4, 135.6)
- moved R3 97.5 mm to (235.7, 135.6)
- moved R4 97.5 mm to (234.5, 135.6)
- moved U5 97.5 mm to (229.1, 137.0)
- moved S1 97.5 mm to (211.8, 149.7)
- moved S2 97.5 mm to (211.8, 131.2)
- moved C1 97.5 mm to (226.8, 154.3)
- moved C2 97.5 mm to (226.2, 147.3)
- moved C3 97.5 mm to (243.9, 148.4)
- moved C4 97.5 mm to (243.4, 154.1)
- moved C8 97.5 mm to (226.2, 140.4)
- moved R1 97.5 mm to (243.9, 150.4)
- moved R2 97.5 mm to (243.9, 152.3)
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Connections:
- U3 pad 1: Net-(U3-Pad1) -> Net-(C9-Pad1)
- U5 pad 2: Net-(U3-Pad1) -> Net-(C9-Pad2)
Routing:
- net Net-(U3-Pad1): track 10.8 -> 0.00 mm
- net GND: track 90.6 -> 101.5 mm
- net Net-(C9-Pad2): track 0.00 -> 8.90 mm
- net +5V: track 71.8 -> 80.1 mm, vias 7 -> 8
- net Net-(C9-Pad1): track 0.00 -> 3.90 mm
- net Net-(S2-PadP): track 20.9 -> 20.8 mm, vias 2 -> 1
