File: Hardware/Sensor/Sensor Completed Project Folder/DCA_USMR_Sens/DCA_USMR_Sens.kicad_sch (KiCad schematic)
At the start: 19 parts, among them U1 LM555xM, U2 MAX4528CSA+, U3 MAX4528CSA+, U4 SN74AHC1G04DBVR, U5 LM193DR

Commit message: Sensor Rev1.1
Rev1.1
Parts:
- added C10: 1u, Capacitor_SMD:C_0402_1005Metric, symbol Device:C_Small
- added C9: 10uF, Capacitor_SMD:C_0402_1005Metric, symbol Device:C_Small
- added D1: 1Vf, DIOAD835W50L444D203:DIOAD835W50L444D203, symbol Device:D_Zener_Small
- added R5: 220, Resistor_SMD:R_0402_1005Metric, symbol Device:R_Small
- R3: value 2.2k -> 2.7k
- R4: value 22k -> 560
Connections:
- net +5V: now also C10.2, R5.1
- net GND: now also C10.1, D1.2 (A)
- net at U5.2 (1IN-): now also C9.2, D1.1 (K), R5.2; no longer U3.1 (A)
- new net: C9.1, U3.1 (A)
Other:
- moved on the sheet: C7
